File: rf.kicad_sch (KiCad schematic)
At the start: 5 parts

Commit message: ERC
Parts:
- gave numbers to parts that had none: 5
Changed lines of the file:
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@@
   (symbol (lib_id "Device:L") (at 95.25 104.775 90) (unit 1)
     (in_bom yes) (on_board yes)
-    (property "Reference" "L?" (id 0) (at 95.25 101.6 90))
+    (property "Reference" "L501" (id 0) (at 95.25 101.6 90))
     (property "Value" "2n7" (id 1) (at 95.25 106.68 90))
     (property "Footprint" "" (id 2) (at 95.25 104.775 0)
@@
   (symbol (lib_id "OxySwitch:748112024") (at 163.83 102.235 0) (mirror y) (unit 1)
     (in_bom yes) (on_board yes) (fields_autoplaced)
-    (property "Reference" "FL?" (id 0) (at 148.59 94.615 0))
+    (property "Reference" "FL501" (id 0) (at 148.59 94.615 0))
     (property "Value" "748112024" (id 1) (at 148.59 97.155 0))
     (property "Footprint" "748112024" (id 2) (at 137.16 99.695 0)
@@
   (symbol (lib_id "power:GND") (at 163.83 98.425 180) (unit 1)
     (in_bom yes) (on_board yes) (fields_autoplaced)
-    (property "Reference" "#PWR?" (id 0) (at 163.83 92.075 0)
+    (property "Reference" "#PWR0505" (id 0) (at 163.83 92.075 0)
       (effects (font (size 1.27 1.27)) hide)
     )
@@
   (symbol (lib_id "power:GND") (at 107.95 117.475 0) (unit 1)
     (in_bom yes) (on_board yes) (fields_autoplaced)
-    (property "Reference" "#PWR?" (id 0) (at 107.95 123.825 0)
+    (property "Reference" "#PWR0502" (id 0) (at 107.95 123.825 0)
       (effects (font (size 1.27 1.27)) hide)
     )
@@
   (symbol (lib_id "Device:C") (at 82.55 111.125 0) (unit 1)
     (in_bom yes) (on_board yes) (fields_autoplaced)
-    (property "Reference" "C?" (id 0) (at 86.36 109.8549 0)
+    (property "Reference" "C501" (id 0) (at 86.36 109.8549 0)
       (effects (font (size 1.27 1.27)) (justify left))
     )
@@
   (symbol (lib_id "power:GND") (at 133.35 98.425 180) (unit 1)
     (in_bom yes) (on_board yes) (fields_autoplaced)
-    (property "Reference" "#PWR?" (id 0) (at 133.35 92.075 0)
+    (property "Reference" "#PWR0503" (id 0) (at 133.35 92.075 0)
       (effects (font (size 1.27 1.27)) hide)
     )
@@
   (symbol (lib_id "power:GND") (at 133.35 111.125 0) (unit 1)
     (in_bom yes) (on_board yes) (fields_autoplaced)
-    (property "Reference" "#PWR?" (id 0) (at 133.35 117.475 0)
+    (property "Reference" "#PWR0504" (id 0) (at 133.35 117.475 0)
       (effects (font (size 1.27 1.27)) hide)
     )
@@
   (symbol (lib_id "power:GND") (at 82.55 117.475 0) (unit 1)
     (in_bom yes) (on_board yes) (fields_autoplaced)
-    (property "Reference" "#PWR?" (id 0) (at 82.55 123.825 0)
+    (property "Reference" "#PWR0501" (id 0) (at 82.55 123.825 0)
       (effects (font (size 1.27 1.27)) hide)
     )
@@
   (symbol (lib_id "power:GND") (at 163.83 111.125 0) (unit 1)
     (in_bom yes) (on_board yes) (fields_autoplaced)
-    (property "Reference" "#PWR?" (id 0) (at 163.83 117.475 0)
+    (property "Reference" "#PWR0506" (id 0) (at 163.83 117.475 0)
       (effects (font (size 1.27 1.27)) hide)
     )
@@
   (symbol (lib_id "Device:C") (at 107.95 111.125 0) (unit 1)
     (in_bom yes) (on_board yes) (fields_autoplaced)
-    (property "Reference" "C?" (id 0) (at 111.76 109.8549 0)
+    (property "Reference" "C502" (id 0) (at 111.76 109.8549 0)
       (effects (font (size 1.27 1.27)) (justify left))
     )
@@
   (symbol (lib_id "OxySwitch:ANT3216LL00R2400A") (at 184.15 104.775 0) (unit 1)
     (in_bom yes) (on_board yes) (fields_autoplaced)
-    (property "Reference" "ANT?" (id 0) (at 200.66 104.7749 0)
+    (property "Reference" "ANT501" (id 0) (at 200.66 104.7749 0)
       (effects (font (size 1.27 1.27)) (justify left))
     )
