File: mcu.kicad_sch (KiCad schematic)
At the start: 11 parts

Commit message: Added RF
Other:
- moved on the sheet: C?, SW?
Changed lines of the file:
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@@
   (junction (at 36.83 177.8) (diameter 0) (color 0 0 0 0)
   )
+  (junction (at 65.405 139.065) (diameter 0) (color 0 0 0 0)
+  )
   (junction (at 17.78 177.8) (diameter 0) (color 0 0 0 0)
   )
   (junction (at 113.03 119.38) (diameter 0) (color 0 0 0 0)
   )
-  (junction (at 69.85 139.7) (diameter 0) (color 0 0 0 0)
+  (junction (at 71.12 139.065) (diameter 0) (color 0 0 0 0)
   )
   (junction (at 62.23 179.07) (diameter 0) (color 0 0 0 0)
@@
     (stroke (width 0) (type default) (color 0 0 0 0))
   )
-  (wire (pts (xy 69.85 149.86) (xy 69.85 152.4))
+  (wire (pts (xy 71.12 149.225) (xy 71.12 151.765))
     (stroke (width 0) (type default) (color 0 0 0 0))
   )
@@
     (stroke (width 0) (type default) (color 0 0 0 0))
   )
-  (wire (pts (xy 69.85 139.7) (xy 69.85 142.24))
+  (wire (pts (xy 71.12 139.065) (xy 71.12 141.605))
     (stroke (width 0) (type default) (color 0 0 0 0))
   )
@@
     (stroke (width 0) (type default) (color 0 0 0 0))
   )
-  (wire (pts (xy 57.15 139.7) (xy 57.15 140.97))
+  (wire (pts (xy 58.42 139.065) (xy 58.42 140.335))
     (stroke (width 0) (type default) (color 0 0 0 0))
   )
@@
     (stroke (width 0) (type default) (color 0 0 0 0))
   )
-  (wire (pts (xy 76.2 139.7) (xy 69.85 139.7))
+  (wire (pts (xy 77.47 139.065) (xy 71.12 139.065))
     (stroke (width 0) (type default) (color 0 0 0 0))
   )
@@
     (stroke (width 0) (type default) (color 0 0 0 0))
   )
+  (wire (pts (xy 65.405 139.065) (xy 58.42 139.065))
+    (stroke (width 0) (type default) (color 0 0 0 0))
+  )
   (wire (pts (xy 179.07 45.72) (xy 184.15 45.72))
     (stroke (width 0) (type default) (color 0 0 0 0))
@@
     (stroke (width 0) (type default) (color 0 0 0 0))
   )
-  (wire (pts (xy 69.85 139.7) (xy 57.15 139.7))
+  (wire (pts (xy 71.12 139.065) (xy 65.405 139.065))
     (stroke (width 0) (type default) (color 0 0 0 0))
   )
@@
     (stroke (width 0) (type default) (color 0 0 0 0))
   )
+  (wire (pts (xy 65.405 139.065) (xy 65.405 141.605))
+    (stroke (width 0) (type default) (color 0 0 0 0))
+  )
   (bus (pts (xy 199.39 116.84) (xy 199.39 121.92))
     (stroke (width 0) (type default) (color 0 0 0 0))
@@
     (stroke (width 0) (type default) (color 0 0 0 0))
   )
-  (wire (pts (xy 57.15 151.13) (xy 57.15 152.4))
+  (wire (pts (xy 58.42 150.495) (xy 58.42 151.765))
     (stroke (width 0) (type default) (color 0 0 0 0))
   )
@@
     )
   )
-  (global_label "NRST" (shape input) (at 76.2 139.7 0) (fields_autoplaced)
-    (effects (font (size 1.27 1.27)) (justify left))
-    (property "Intersheet References" "${INTERSHEET_REFS}" (id 0) (at 83.3907 139.6206 0)
+  (global_label "NRST" (shape input) (at 77.47 139.065 0) (fields_autoplaced)
+    (effects (font (size 1.27 1.27)) (justify left))
+    (property "Intersheet References" "${INTERSHEET_REFS}" (id 0) (at 84.6607 138.9856 0)
       (effects (font (size 1.27 1.27)) (justify left) hide)
     )
@@
     (effects (font (size 1.27 1.27)) (justify right))
   )
+  (hierarchical_label "NRST" (shape input) (at 65.405 141.605 270)
+    (effects (font (size 1.27 1.27)) (justify right))
+  )
   (hierarchical_label "RF1" (shape input) (at 184.15 71.12 0)
     (effects (font (size 1.27 1.27)) (justify left))
@@
     (pin "1")
   )
-  (symbol (lib_id "Device:C") (at 69.85 146.05 0) (unit 1)
-    (in_bom yes) (on_board yes) (fields_autoplaced)
-    (property "Reference" "C?" (id 0) (at 72.771 145.2153 0)
+  (symbol (lib_id "Device:C") (at 71.12 145.415 0) (unit 1)
+    (in_bom yes) (on_board yes) (fields_autoplaced)
+    (property "Reference" "C?" (id 0) (at 74.041 144.5803 0)
       (effects (font (size 1.27 1.27)) (justify left))
     )
-    (property "Value" "C" (id 1) (at 72.771 147.7522 0)
+    (property "Value" "C" (id 1) (at 74.041 147.1172 0)
       (effects (font (size 1.27 1.27)) (justify left))
     )
-    (property "Footprint" "" (id 2) (at 70.8152 149.86 0)
-      (effects (font (size 1.27 1.27)) hide)
-    )
-    (property "Datasheet" "~" (id 3) (at 69.85 146.05 0)
+    (property "Footprint" "" (id 2) (at 72.0852 149.225 0)
+      (effects (font (size 1.27 1.27)) hide)
+    )
+    (property "Datasheet" "~" (id 3) (at 71.12 145.415 0)
       (effects (font (size 1.27 1.27)) hide)
     )
@@
     (pin "2")
   )
-  (symbol (lib_id "Switch:SW_Push") (at 57.15 146.05 90) (unit 1)
-    (in_bom yes) (on_board yes) (fields_autoplaced)
-    (property "Reference" "SW?" (id 0) (at 58.293 146.4838 90)
+  (symbol (lib_id "Switch:SW_Push") (at 58.42 145.415 90) (unit 1)
+    (in_bom yes) (on_board yes) (fields_autoplaced)
+    (property "Reference" "SW?" (id 0) (at 59.563 145.8488 90)
       (effects (font (size 1.27 1.27)) (justify right))
     )
-    (property "Value" "SW_Push" (id 1) (at 58.293 147.7522 90)
+    (property "Value" "SW_Push" (id 1) (at 59.563 147.1172 90)
       (effects (font (size 1.27 1.27)) (justify right) hide)
     )
-    (property "Footprint" "" (id 2) (at 52.07 146.05 0)
-      (effects (font (size 1.27 1.27)) hide)
-    )
-    (property "Datasheet" "~" (id 3) (at 52.07 146.05 0)
+    (property "Footprint" "" (id 2) (at 53.34 145.415 0)
+      (effects (font (size 1.27 1.27)) hide)
+    )
+    (property "Datasheet" "~" (id 3) (at 53.34 145.415 0)
       (effects (font (size 1.27 1.27)) hide)
     )
@@
     (pin "1")
   )
-  (symbol (lib_id "power:GND") (at 57.15 152.4 0) (unit 1)
-    (in_bom yes) (on_board yes) (fields_autoplaced)
-    (property "Reference" "#PWR?" (id 0) (at 57.15 158.75 0)
-      (effects (font (size 1.27 1.27)) hide)
-    )
-    (property "Value" "GND" (id 1) (at 57.15 156.8434 0))
-    (property "Footprint" "" (id 2) (at 57.15 152.4 0)
-      (effects (font (size 1.27 1.27)) hide)
-    )
-    (property "Datasheet" "" (id 3) (at 57.15 152.4 0)
+  (symbol (lib_id "power:GND") (at 58.42 151.765 0) (unit 1)
+    (in_bom yes) (on_board yes) (fields_autoplaced)
+    (property "Reference" "#PWR?" (id 0) (at 58.42 158.115 0)
+      (effects (font (size 1.27 1.27)) hide)
+    )
+    (property "Value" "GND" (id 1) (at 58.42 156.2084 0))
+    (property "Footprint" "" (id 2) (at 58.42 151.765 0)
+      (effects (font (size 1.27 1.27)) hide)
+    )
+    (property "Datasheet" "" (id 3) (at 58.42 151.765 0)
       (effects (font (size 1.27 1.27)) hide)
     )
@@
     (pin "2")
   )
-  (symbol (lib_id "power:GND") (at 69.85 152.4 0) (unit 1)
-    (in_bom yes) (on_board yes) (fields_autoplaced)
-    (property "Reference" "#PWR?" (id 0) (at 69.85 158.75 0)
-      (effects (font (size 1.27 1.27)) hide)
-    )
-    (property "Value" "GND" (id 1) (at 69.85 156.8434 0))
-    (property "Footprint" "" (id 2) (at 69.85 152.4 0)
-      (effects (font (size 1.27 1.27)) hide)
-    )
-    (property "Datasheet" "" (id 3) (at 69.85 152.4 0)
-      (effects (font (size 1.27 1.27)) hide)
-    )
+  (symbol (lib_id "power:GND") (at 71.12 151.765 0) (unit 1)
+    (in_bom yes) (on_board yes) (fields_autoplaced)
+    (property "Reference" "#PWR?" (id 0) (at 71.12 158.115 0)
+      (effects (font (size 1.27 1.27)) hide)
+    )
+    (property "Value" "GND" (id 1) (at 71.12 156.2084 0))
+    (property "Footprint" "" (id 2) (at 71.12 151.765 0)
+      (effects (font (size 1.27 1.27)) hide)
+    )
+    (property "Datasheet" "" (id 3) (at 71.12 151.765 0)
+      (effects (font (size 1.27 1.27)) hide)
+    )

Commit message: ERC
Parts:
- gave numbers to parts that had none: 11
Connections:
- no-connect marks 0 -> 27
Other:
- moved on the sheet: SW201

Commit message: Schematic cleanup
Changed lines of the file:
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@@
     (company "Tomas Kysela")
   )
+  (bus_alias "SWD" (members "SWDIO" "SWCLCK"))
   (bus_alias "VDD" (members "VDDA" "VDDRF" "VDDUSB" "VDDSMPS" "VDD1" "VDD2" "VDD3"))
-  (bus_alias "SWD" (members "SWDIO" "SWCLCK"))
   (junction (at 36.83 177.8) (diameter 0) (color 0 0 0 0)
   )
@@
     )
   )
-  (global_label "NRST" (shape input) (at 77.47 139.065 0) (fields_autoplaced)
+  (global_label "NRST" (shape output) (at 77.47 139.065 0) (fields_autoplaced)
     (effects (font (size 1.27 1.27)) (justify left))
     (property "Intersheet References" "${INTERSHEET_REFS}" (id 0) (at 84.6607 138.9856 0)
@@
     )
   )
-  (global_label "OSC_OUT" (shape input) (at 184.15 83.82 0) (fields_autoplaced)
-    (effects (font (size 1.27 1.27)) (justify left))
-    (property "Intersheet References" "${INTERSHEET_REFS}" (id 0) (at 194.9693 83.8994 0)
+  (global_label "OSC_OUT" (shape output) (at 184.15 83.82 0) (fields_autoplaced)
+    (effects (font (size 1.27 1.27)) (justify left))
+    (property "Intersheet References" "${INTERSHEET_REFS}" (id 0) (at 194.9693 83.7406 0)
       (effects (font (size 1.27 1.27)) (justify left) hide)
     )
@@
     )
   )
-  (global_label "VFBSMPS" (shape input) (at 184.15 124.46 0) (fields_autoplaced)
-    (effects (font (size 1.27 1.27)) (justify left))
-    (property "Intersheet References" "${INTERSHEET_REFS}" (id 0) (at 195.1507 124.5394 0)
+  (global_label "VFBSMPS" (shape output) (at 184.15 124.46 0) (fields_autoplaced)
+    (effects (font (size 1.27 1.27)) (justify left))
+    (property "Intersheet References" "${INTERSHEET_REFS}" (id 0) (at 195.1507 124.3806 0)
       (effects (font (size 1.27 1.27)) (justify left) hide)
     )
@@
     )
   )
-  (global_label "OSC32_IN" (shape input) (at 36.83 174.625 90) (fields_autoplaced)
+  (global_label "OSC32_IN" (shape output) (at 36.83 174.625 90) (fields_autoplaced)
     (effects (font (size 1.27 1.27)) (justify left))
     (property "Intersheet References" "${INTERSHEET_REFS}" (id 0) (at 36.7506 163.08 90)
@@
     )
   )
-  (global_label "OSC32_OUT" (shape input) (at 184.15 48.26 0) (fields_autoplaced)
+  (global_label "OSC32_OUT" (shape output) (at 184.15 48.26 0) (fields_autoplaced)
     (effects (font (size 1.27 1.27)) (justify left))
     (property "Intersheet References" "${INTERSHEET_REFS}" (id 0) (at 197.3883 48.1806 0)
@@
     )
   )
-  (global_label "PH3-BOOT0" (shape input) (at 102.235 187.96 180) (fields_autoplaced)
+  (global_label "PH3-BOOT0" (shape output) (at 102.235 187.96 180) (fields_autoplaced)
     (effects (font (size 1.27 1.27)) (justify right))
     (property "Intersheet References" "${INTERSHEET_REFS}" (id 0) (at 88.3314 187.8806 0)
@@
     )
   )
-  (global_label "VLXSMPS" (shape input) (at 184.15 129.54 0) (fields_autoplaced)
-    (effects (font (size 1.27 1.27)) (justify left))
-    (property "Intersheet References" "${INTERSHEET_REFS}" (id 0) (at 195.0298 129.6194 0)
-      (effects (font (size 1.27 1.27)) (justify left) hide)
-    )
-  )
-  (global_label "OSC_IN" (shape input) (at 38.1 146.05 0) (fields_autoplaced)
+  (global_label "VLXSMPS" (shape output) (at 184.15 129.54 0) (fields_autoplaced)
+    (effects (font (size 1.27 1.27)) (justify left))
+    (property "Intersheet References" "${INTERSHEET_REFS}" (id 0) (at 195.0298 129.4606 0)
+      (effects (font (size 1.27 1.27)) (justify left) hide)
+    )
+  )
+  (global_label "OSC_IN" (shape output) (at 38.1 146.05 0) (fields_autoplaced)
     (effects (font (size 1.27 1.27)) (justify left))
     (property "Intersheet References" "${INTERSHEET_REFS}" (id 0) (at 47.226 145.9706 0)
@@
     (effects (font (size 1.27 1.27)) (justify left))
   )
-  (hierarchical_label "{SWD}" (shape input) (at 96.52 83.82 180)
+  (hierarchical_label "{SWD}" (shape output) (at 96.52 83.82 180)
     (effects (font (size 1.27 1.27)) (justify right))
   )
@@
     (effects (font (size 1.27 1.27)) (justify right))
   )
-  (hierarchical_label "RF1" (shape input) (at 184.15 71.12 0)
-    (effects (font (size 1.27 1.27)) (justify left))
-  )
+  (hierarchical_label "RF1" (shape output) (at 184.15 71.12 0)
+    (effects (font (size 1.27 1.27)) (justify left))
+  )
