File: zero_detect.kicad_sch (KiCad schematic)
At the start: 6 parts

Commit message: Finished basic version
Parts:
- gave numbers to parts that had none: 6
Changed lines of the file:
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@@
   (symbol (lib_id "OxySwitch:RH06-T") (at 120.65 107.95 0) (unit 1)
     (in_bom yes) (on_board yes) (fields_autoplaced)
-    (property "Reference" "BR?" (id 0) (at 132.08 101.761 0))
+    (property "Reference" "BR701" (id 0) (at 132.08 101.761 0))
     (property "Value" "RH06-T" (id 1) (at 132.08 104.2979 0))
     (property "Footprint" "SOP250P700X300-4N" (id 2) (at 139.7 105.41 0)
@@
   (symbol (lib_id "power:GND") (at 185.42 114.3 0) (unit 1)
     (in_bom yes) (on_board yes) (fields_autoplaced)
-    (property "Reference" "#PWR?" (id 0) (at 185.42 120.65 0)
+    (property "Reference" "#PWR0702" (id 0) (at 185.42 120.65 0)
       (effects (font (size 1.27 1.27)) hide)
     )
@@
   (symbol (lib_id "Device:R") (at 185.42 102.87 0) (unit 1)
     (in_bom yes) (on_board yes) (fields_autoplaced)
-    (property "Reference" "R?" (id 0) (at 187.198 102.0353 0)
+    (property "Reference" "R703" (id 0) (at 187.198 102.0353 0)
       (effects (font (size 1.27 1.27)) (justify left))
     )
@@
   (symbol (lib_id "Device:R") (at 107.95 114.3 90) (unit 1)
     (in_bom yes) (on_board yes)
-    (property "Reference" "R?" (id 0) (at 107.95 111.76 90))
+    (property "Reference" "R702" (id 0) (at 107.95 111.76 90))
     (property "Value" "47k" (id 1) (at 107.95 116.84 90))
     (property "Footprint" "" (id 2) (at 107.95 116.078 90)
@@
   (symbol (lib_id "Device:R") (at 198.12 102.87 0) (unit 1)
     (in_bom yes) (on_board yes) (fields_autoplaced)
-    (property "Reference" "R?" (id 0) (at 199.898 102.0353 0)
+    (property "Reference" "R704" (id 0) (at 199.898 102.0353 0)
       (effects (font (size 1.27 1.27)) (justify left))
     )
@@
   (symbol (lib_id "OxySwitch:MCT2ESM") (at 152.4 107.95 0) (unit 1)
     (in_bom yes) (on_board yes) (fields_autoplaced)
-    (property "Reference" "Q?" (id 0) (at 163.83 101.761 0))
+    (property "Reference" "Q701" (id 0) (at 163.83 101.761 0))
     (property "Value" "MCT2ESM" (id 1) (at 163.83 104.2979 0))
     (property "Footprint" "SOT254P916X480-6N" (id 2) (at 171.45 105.41 0)
@@
   (symbol (lib_id "power:GND") (at 185.42 96.52 180) (unit 1)
     (in_bom yes) (on_board yes) (fields_autoplaced)
-    (property "Reference" "#PWR?" (id 0) (at 185.42 90.17 0)
+    (property "Reference" "#PWR0701" (id 0) (at 185.42 90.17 0)
       (effects (font (size 1.27 1.27)) hide)
     )
@@
   (symbol (lib_id "Device:R") (at 107.95 104.14 90) (unit 1)
     (in_bom yes) (on_board yes)
-    (property "Reference" "R?" (id 0) (at 107.95 101.6 90))
+    (property "Reference" "R701" (id 0) (at 107.95 101.6 90))
     (property "Value" "47k" (id 1) (at 107.95 106.68 90))
     (property "Footprint" "" (id 2) (at 107.95 105.918 90)
